Commit message: Add RRT*, refer to branch RobotArms_Prototype_modified; fix touching_ground_check bugs; fix self_collision bugs

File: assets/ur5e/_ur5e.urdf (robot description, URDF)
Before this commit: robot ur5e, 11 links, 10 joints
Links:
- link base_link: geometry collision mesh filename=package://ur5e/meshes/collision/base.stl scale=1.0 1.0 1.0; visual mesh filename=package://ur5e/meshes/visual/base.dae
- link forearm_link: geometry collision mesh filename=package://ur5e/meshes/collision/forearm.stl scale=1.0 1.0 1.0; visual mesh filename=package://ur5e/meshes/visual/forearm.dae
- link shoulder_link: geometry collision mesh filename=package://ur5e/meshes/collision/shoulder.stl scale=1.0 1.0 1.0; visual mesh filename=package://ur5e/meshes/visual/shoulder.dae
- link upper_arm_link: geometry collision mesh filename=package://ur5e/meshes/collision/upperarm.stl scale=1.0 1.0 1.0; visual mesh filename=package://ur5e/meshes/visual/upperarm.dae
- link wrist_1_link: geometry collision mesh filename=package://ur5e/meshes/collision/wrist1.stl scale=1.0 1.0 1.0; visual mesh filename=package://ur5e/meshes/visual/wrist1.dae
- link wrist_2_link: geometry collision mesh filename=package://ur5e/meshes/collision/wrist2.stl scale=1.0 1.0 1.0; visual mesh filename=package://ur5e/meshes/visual/wrist2.dae
- link wrist_3_link: geometry collision mesh filename=package://ur5e/meshes/collision/wrist3.stl scale=1.0 1.0 1.0; visual mesh filename=package://ur5e/meshes/visual/wrist3.dae
